Commit message: Add gen_convex_stl.py & gen_srdf.py

File: mani_skill/assets/robots/fetch/fetch_torso_up.urdf (robot description, URDF)
Before this commit: robot fetch, 20 links, 19 joints
Joints:
- joint forearm_roll_joint: limit effort=29.35 velocity=1.571 -> lower=-3.142 upper=3.142 effort=29.35 velocity=1.571; type continuous -> revolute
- joint upperarm_roll_joint: limit effort=76.94 velocity=1.571 -> lower=-3.142 upper=3.142 effort=76.94 velocity=1.571; type continuous -> revolute
- joint wrist_roll_joint: limit effort=7.36 velocity=2.268 -> lower=-3.142 upper=3.142 effort=7.36 velocity=2.268; type continuous -> revolute
